File: Arm_Main.kicad_pcb (KiCad board)
At the start: 2 copper layers, 100 x 110 mm, 33 parts, among them IC1 TLP559_F_, J1 Conn_01x03_Socket, J2 Conn_01x02_Pin, J4 Conn_01x03_Pin, J5 Conn_01x03_Pin, J6 Conn_01x03_Pin, SW2 SW_SPDT, U1 RASPBERRY_PI_ZERO_2_W, U2 TLP2531, U3 TLP2531

Commit message: ver5
Other:
- board text added: "ARM_Main_ver5"
- board text removed: "ARM_Main_ver4"
Changed lines of the file:
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@@
 		(layer "Edge.Cuts")
 	)
-	(gr_text "ARM_Main_ver4"
+	(gr_text "ARM_Main_ver5"
 		(at 158.6 42.6 0)
 		(layer "F.SilkS")
