File: Arm_Main.kicad_pcb (KiCad board)
At the start: 2 copper layers, 100 x 110 mm, 33 parts, among them IC1 TLP559_F_, J1 Conn_01x03_Socket, J2 Conn_01x02_Pin, J4 Conn_01x03_Pin, J5 Conn_01x03_Pin, J6 Conn_01x03_Pin, SW2 SW_SPDT, U1 RASPBERRY_PI_ZERO_2_W, U2 TLP2531, U3 TLP2531

Commit message: ver6
Connections:
- SB1 pad 7: Net-(SB1-G) -> Net-(SB1-G')
- SB1 pad 8: Net-(D3-K) -> Net-(SB1-Vcc)
- U1 pad 1: unconnected-(U1-3V3_1-Pad1) -> Net-(SB1-Vcc)
- U1 pad 12: Net-(SB1-G) -> Net-(SB1-G')
- U1 pad 15: Net-(SB1-G') -> unconnected-(U1-GPIO22/GPIO_GEN3-Pad15)
Routing:
- net Net-(SB1-Vcc): track 0.00 -> 50.6 mm, vias 0 -> 3
- net Net-(SB1-G): track 38.0 -> 0.00 mm
- net Net-(D3-K): track 151.4 -> 147.4 mm
- net Net-(SB1-G'): track 41.7 -> 44.8 mm
- net GNDA: vias 201 -> 222
Other:
- board text added: "ARM_Main_ver6"
- board text removed: "ARM_Main_ver5"
