File: Arm_Main.kicad_pcb (KiCad board)
At the start: 2 copper layers, 100 x 110 mm, 33 parts, among them IC1 TLP559_F_, J1 Conn_01x03_Socket, J2 Conn_01x02_Pin, J4 Conn_01x03_Pin, J5 Conn_01x03_Pin, J6 Conn_01x03_Pin, SW2 SW_SPDT, U1 RASPBERRY_PI_ZERO_2_W, U2 TLP2531, U3 TLP2531

Commit message: Ver_7
Parts:
- removed J6: Conn_01x03_Pin, Connector_PinHeader_2.54mm:PinHeader_1x03_P2.54mm_Vertical
- removed SW2: SW_SPDT, Togle_original:TogleSW3pin
- added D5: LED, LED_THT:LED_D3.0mm, F.Cu at (153.6, 120.9)
- added J3: Conn_01x03_Pin, Connector_PinHeader_2.54mm:PinHeader_1x03_P2.54mm_Vertical, F.Cu at (162.1, 129.4)
- added R7: 1k, Resistor_THT:R_Axial_DIN0207_L6.3mm_D2.5mm_P10.16mm_Horizontal, F.Cu at (153.6, 105.4)
- added SW1: SW_SPDT, Togle_original:TogleSW3pin, F.Cu at (124.1, 98.4)
- C3: value 0.1u -> 100u; footprint Capacitor_THT:C_Disc_D5.1mm_W3.2mm_P5.00mm -> Capacitor_THT:CP_Radial_D5.0mm_P2.50mm
- C4: value 100u -> 0.1u; footprint Capacitor_THT:CP_Radial_D5.0mm_P2.50mm -> Capacitor_THT:C_Disc_D5.1mm_W3.2mm_P5.00mm
- C6: value 0.1u -> 47u; footprint Capacitor_THT:C_Disc_D5.1mm_W3.2mm_P5.00mm -> Capacitor_THT:CP_Radial_D5.0mm_P2.50mm
- C7: value 47u -> 0.1u; footprint Capacitor_THT:CP_Radial_D5.0mm_P2.50mm -> Capacitor_THT:C_Disc_D5.1mm_W3.2mm_P5.00mm
- J1: value Conn_01x03_Socket -> Conn_01x02_Pin; footprint Connector_JST:JST_XH_B3B-XH-A_1x03_P2.50mm_Vertical -> Connector_AMASS:AMASS_XT30U-F_1x02_P5.0mm_Vertical
- J2: value Conn_01x02_Pin -> Conn_01x03_Pin; footprint Connector_AMASS:AMASS_XT30U-F_1x02_P5.0mm_Vertical -> Connector_PinHeader_2.54mm:PinHeader_1x03_P2.54mm_Vertical
- J5: value Conn_01x03_Pin -> Conn_01x03_Socket; footprint Connector_PinHeader_2.54mm:PinHeader_1x03_P2.54mm_Vertical -> Connector_JST:JST_XH_B3B-XH-A_1x03_P2.50mm_Vertical
- R1: value 20k -> 2k
- R2: value 1.2k -> 20k
- R4: value 2k -> 1.2k
- RV1, RV2: value R_Potentiometer_Trim -> R_Trim
- U3: value TLP2531 -> ADuM121N; footprint ul_TLP2531:U_DIP8_11-10C4S_TOS -> Package_SO:SOIC-8_3.9x4.9mm_P1.27mm
- VR1: footprint NJM317:TO254P1054X470X1955-3 -> Njm317_original:TO254P1054X470X1955-3
- moved J2 88.6 mm to (165.8, 129.4), turned to 180 degrees
- moved U2 68.3 mm to (164.9, 104.2)
- moved D1 64.9 mm to (151.1, 98.7), turned to 180 degrees
- moved SB1 58.5 mm to (163.4, 89.6), turned to 180 degrees
- moved J5 42.3 mm to (151.5, 82.4), turned to 0 degrees
- moved J1 40.3 mm to (120.3, 89.8), turned to 0 degrees
- moved R3 38.6 mm to (133.6, 62.6), turned to -90 degrees
- moved C1 37.2 mm to (134.5, 91.4), turned to 0 degrees
- moved RV1 36.7 mm to (143.4, 72.9), turned to 90 degrees
- moved D2 34.8 mm to (122.5, 84.4)
- moved R1 34.1 mm to (134.5, 98.7), turned to 0 degrees
- moved R2 33.7 mm to (134.5, 95.1), turned to 0 degrees
- moved R6 32.3 mm to (148.5, 115.6)
- moved U1 30.4 mm to (183.1, 98.6)
- moved IC1 30.0 mm to (161.4, 114.1)
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Connections:
- C1 pad 1: Net-(D3-K) -> Batte
- C2 pad 1: Net-(MD1-SENSE) -> +5V_Digital
- C3 pad 1: Net-(D3-K) -> Batte
- C4 pad 1: Net-(D3-K) -> Batte
- C6 pad 1: Net-(D3-A) -> +5V_Analog
- C7 pad 1: Net-(D3-A) -> +5V_Analog
- D3 pad 1: Net-(D3-K) -> Batte
- D3 pad 2: Net-(D3-A) -> +5V_Analog
- D4 pad 1: Net-(D3-A) -> +5V_Analog
- IC1 pad 8: Net-(D3-K) -> Batte
- J1 pad 1: Net-(D3-K) -> GNDA
- J2 pad 1: GNDA -> +5V_Analog
- J2 pad 2: +BATT -> Net-(J2-Pin_2)
- J4 pad 1: Net-(D3-A) -> +5V_Analog
- J4 pad 2: Net-(J4-Pin_2) -> Net-(IC1-COLLECTER)
- J5 pad 1: Net-(D3-A) -> Batte
- MD1 pad 2: Net-(D3-K) -> Batte
- MD1 pad 4: Net-(MD1-SENSE) -> +5V_Digital
- MD1 pad 5: Net-(MD1-SENSE) -> +5V_Digital
- R1 pad 1: Net-(D3-K) -> Batte
- R1 pad 2: GNDA -> Net-(D1-A)
- R2 pad 1: Net-(MD1-SENSE) -> Batte
- R4 pad 1: Net-(D3-K) -> +5V_Digital
- R4 pad 2: Net-(D1-A) -> GNDA
- R5 pad 1: Net-(MD1-SENSE) -> +5V_Digital
- R6 pad 2: Net-(D3-A) -> +5V_Analog
- U1 pad 12: Net-(SB1-G') -> Net-(SB1-A1)
- U1 pad 13: Net-(SB1-A1) -> Net-(SB1-G')
- U1 pad 17: unconnected-(U1-3V3_17-Pad17) -> Net-(SB1-Vcc)
- U1 pad 2: Net-(MD1-SENSE) -> +5V_Digital
- U1 pad 4: unconnected-(U1-5V_4-Pad4) -> +5V_Digital
- U2 pad 1: Net-(SB1-A2) -> Net-(U1-GPIO24/GPIO_GEN5)
- U2 pad 4: Net-(J1-Pin_2) -> Net-(U1-GPIO23/GPIO_GEN4)
- U2 pad 6: Net-(SB1-A2) -> Net-(J2-Pin_2)
- U2 pad 7: Net-(J1-Pin_2) -> Net-(J3-Pin_2)
- U2 pad 8: Net-(D3-K) -> Batte
- U3 pad 1: Net-(U1-GPIO23/GPIO_GEN4) -> Net-(SB1-Vcc)
- U3 pad 2: GNDA -> Net-(SB1-A2)
- U3 pad 3: GNDA -> Net-(SB1-A2)
- U3 pad 4: Net-(U1-GPIO24/GPIO_GEN5) -> GNDA
- U3 pad 6: Net-(J4-Pin_2) -> Net-(J5-Pin_2)
- U3 pad 8: Net-(D3-K) -> +5V_Analog
- VR1 pad 2: Net-(D3-A) -> +5V_Analog
- VR1 pad 3: Net-(D3-K) -> Batte
Routing:
- net GNDA: track 525.8 -> 280.8 mm, vias 222 -> 239
- net Net-(D3-K): track 147.4 -> 0.00 mm, vias 4 -> 0
- net Batte: track 0.00 -> 113.7 mm
- net Net-(D3-A): track 108.9 -> 0.00 mm, vias 4 -> 0
- net +5V_Analog: track 0.00 -> 89.3 mm, vias 0 -> 1
- net Net-(MD1-SENSE): track 60.5 -> 0.00 mm, vias 3 -> 0
- net +5V_Digital: track 0.00 -> 57.1 mm
- net Net-(J4-Pin_2): track 39.0 -> 0.00 mm
- net Net-(SB1-A1): track 40.0 -> 6.59 mm
- net Net-(SB1-G'): track 44.8 -> 12.2 mm
- net Net-(J2-Pin_2): track 0.00 -> 32.4 mm
- net Net-(J5-Pin_2): track 41.1 -> 10.6 mm
- net Net-(J3-Pin_2): track 0.00 -> 28.3 mm
- net Net-(J1-Pin_2): track 29.3 -> 9.10 mm
- net Net-(IC1-COLLECTER): track 35.4 -> 15.7 mm
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Other:
- board size 100 x 110 mm -> 99 x 78.5 mm
- board text added: "ARM_Main_Ver7"
- board text removed: "ARM_Main_ver6"

Commit message: ver.8.pre
Parts:
- removed SW1: SW_SPDT, Togle_original:TogleSW3pin
- added C10: 1000u, Capacitor_THT:CP_Radial_D10.0mm_P5.00mm, F.Cu at (126.8, 62.1)
- added C8: 0.1u, Capacitor_THT:C_Disc_D5.1mm_W3.2mm_P5.00mm, F.Cu at (11.7, 115.2)
- added C9: 0.1u, Capacitor_THT:C_Disc_D5.1mm_W3.2mm_P5.00mm, F.Cu at (11.7, 120.0)
- added IC2: TLP559_F_, TLP559:DIP762W60P254L966H485Q8N, F.Cu at (56.5, 111.9)
- added SW4: SW_SPST, Togle_original:Hadou_Sw, F.Cu at (18.7, 70.2)
- added SW5: SW_SPST, Togle_original:Hadou_Sw, F.Cu at (18.7, 79.7)
- added SW6: SW_SPST, Togle_original:Hadou_Sw, F.Cu at (126.1, 73.5)
- RV1: moved to B.Cu
- moved U2 136.5 mm to (28.8, 113.7), turned to 0 degrees
- moved J2 127.6 mm to (54.2, 67.6), turned to 0 degrees
- moved R7 124.8 mm to (28.8, 109.8), turned to 0 degrees
- moved C5 122.5 mm to (20.4, 103.7)
- moved C7 120.7 mm to (11.7, 110.5), turned to 0 degrees
- moved J3 120.4 mm to (58.8, 67.6), turned to 0 degrees
- moved R6 120.1 mm to (28.8, 105.7), turned to 0 degrees
- moved C6 116.0 mm to (20.4, 110.2)
- moved C4 115.6 mm to (11.7, 105.7), turned to 0 degrees
- moved IC1 115.5 mm to (45.9, 111.9), turned to 0 degrees
- moved J4 113.4 mm to (63.3, 67.6), turned to 0 degrees
- moved RV2 107.2 mm to (42.5, 103.0), turned to 0 degrees
- moved U3 103.7 mm to (56.9, 121.0), turned to 0 degrees
- moved C3 102.7 mm to (20.4, 97.1), turned to 0 degrees
- moved D5 95.9 mm to (67.3, 79.0), turned to 0 degrees
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Connections:
- IC1 pad 8: Batte -> +5V_Analog
- J2 pad 1: +5V_Analog -> Net-(J2-Pin_1)
- J3 pad 1: +5V_Analog -> Net-(J2-Pin_1)
- J4 pad 1: +5V_Analog -> Net-(J2-Pin_1)
- J5 pad 1: Batte -> Net-(J5-Pin_1)
- SB1 pad 1: Net-(SB1-G') -> Net-(IC2-COLLECTER)
- SB1 pad 3: Net-(SB1-A1) -> Net-(SB1-Y2)
- SB1 pad 5: Net-(SB1-A2) -> Net-(J5-Pin_2)
- SB1 pad 6: Net-(SB1-A2) -> Net-(J5-Pin_2)
- SB1 pad 7: Net-(SB1-G') -> Net-(IC2-COLLECTER)
- SB1 pad 8: Net-(SB1-Vcc) -> +5V_Analog
- U1 pad 1: Net-(SB1-Vcc) -> Net-(U1-3V3_1)
- U1 pad 10: unconnected-(U1-GPIO15/RXD0-Pad10) -> Net-(U1-GPIO15/RXD0)
- U1 pad 12: Net-(SB1-A1) -> unconnected-(U1-GPIO18/GPIO_GEN1-Pad12)
- U1 pad 13: Net-(SB1-G') -> unconnected-(U1-GPIO27/GPIO_GEN2-Pad13)
- U1 pad 17: Net-(SB1-Vcc) -> Net-(U1-3V3_1)
- U1 pad 36: unconnected-(U1-GPIO16-Pad36) -> Net-(IC2-ANODE)
- U1 pad 8: unconnected-(U1-GPIO14/TXD0-Pad8) -> Net-(U1-GPIO14/TXD0)
- U2 pad 8: Batte -> +5V_Analog
- U3 pad 1: Net-(SB1-Vcc) -> Net-(U1-3V3_1)
- U3 pad 2: Net-(SB1-A2) -> Net-(U1-GPIO15/RXD0)
- U3 pad 3: Net-(SB1-A2) -> Net-(U1-GPIO14/TXD0)
- U3 pad 6: Net-(J5-Pin_2) -> Net-(SB1-A1)
- U3 pad 7: Net-(J5-Pin_2) -> Net-(SB1-Y2)
Routing:
- net GNDA: track 280.8 -> 0.00 mm, vias 239 -> 0
- net Batte: track 113.7 -> 0.00 mm
- net +5V_Analog: track 89.3 -> 0.00 mm, vias 1 -> 0
- net +5V_Digital: track 57.1 -> 0.00 mm
- net Net-(SB1-Vcc): track 52.8 -> 0.00 mm, vias 1 -> 0
- net Net-(J2-Pin_2): track 32.4 -> 0.00 mm
- net Net-(D4-A): track 31.1 -> 0.00 mm
- net Net-(J3-Pin_2): track 28.3 -> 0.00 mm
- net Net-(IC1-ANODE): track 17.6 -> 0.00 mm
- net Net-(IC1-COLLECTER): track 15.7 -> 0.00 mm
- net Net-(SB1-G'): track 12.2 -> 0.00 mm
- net Net-(U1-GPIO24/GPIO_GEN5): track 11.7 -> 0.00 mm
- net Net-(J5-Pin_2): track 10.6 -> 0.00 mm
- net Net-(J1-Pin_2): track 9.10 -> 0.00 mm
- net Net-(MD1-TRIM): track 8.00 -> 0.00 mm, vias 1 -> 0
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- removed copper zone on B.Cu, net GNDA
- removed copper zone on F.Cu, net GNDA
Other:
- outline, holes or cut-outs redrawn
- board text added: "ARM_Main_Ver8"
- board text removed: "ARM_Main_Ver7"

Commit message: v8.1
Parts:
- RV1: moved to F.Cu
- moved C8 173.9 mm to (178.1, 64.6)
- moved C9 172.0 mm to (178.1, 76.4)
- moved U2 133.7 mm to (162.4, 108.4), turned to -90 degrees
- moved U3 133.5 mm to (180.5, 70.6), turned to 90 degrees
- moved SW5 131.8 mm to (146.0, 113.8), turned to -90 degrees
- moved SW4 128.7 mm to (147.3, 66.1), turned to -90 degrees
- moved C5 117.0 mm to (137.4, 103.8), turned to 90 degrees
- moved J4 116.5 mm to (164.3, 125.9), turned to 180 degrees
- moved J3 116.2 mm to (159.3, 125.9), turned to 180 degrees
- moved J2 116.1 mm to (154.6, 125.9), turned to 180 degrees
- moved R7 114.8 mm to (142.5, 93.9), turned to -90 degrees
- moved IC1 113.3 mm to (158.6, 100.2), turned to -90 degrees
- moved IC2 109.2 mm to (158.9, 74.0), turned to 180 degrees
- moved C7 108.7 mm to (120.1, 101.2)
- moved J5 108.6 mm to (155.7, 60.9)
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Connections:
- U1 pad 12: unconnected-(U1-GPIO18/GPIO_GEN1-Pad12) -> Net-(IC2-ANODE)
- U1 pad 36: Net-(IC2-ANODE) -> unconnected-(U1-GPIO16-Pad36)
Routing:
- net +5V_Analog: track 0.00 -> 166.3 mm, vias 0 -> 4
- net Batte: track 0.00 -> 95.5 mm
- net GNDA: track 0.00 -> 93.5 mm, vias 0 -> 153
- net +5V_Digital: track 0.00 -> 67.2 mm, vias 0 -> 1
- net Net-(U1-3V3_1): track 0.00 -> 37.7 mm
- net Net-(U1-GPIO23/GPIO_GEN4): track 0.00 -> 34.4 mm
- net Net-(SB1-A1): track 0.00 -> 31.0 mm
- net Net-(J2-Pin_1): track 0.00 -> 26.9 mm
- net Net-(IC1-COLLECTER): track 0.00 -> 26.7 mm
- net Net-(D4-A): track 0.00 -> 24.1 mm
- net Net-(SB1-Y2): track 0.00 -> 22.7 mm
- net Net-(U1-GPIO24/GPIO_GEN5): track 0.00 -> 21.8 mm
- net Net-(IC2-ANODE): track 0.00 -> 19.7 mm, vias 0 -> 1
- net Net-(U1-GPIO14/TXD0): track 0.00 -> 18.2 mm
- net Net-(U1-GPIO15/RXD0): track 0.00 -> 13.1 mm
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- added copper zone on B.Cu, net GNDA
- added copper zone on F.Cu, net GNDA
Other:
- outline, holes or cut-outs redrawn
- board text added: "ARM_Main_Ver8.1"
- board text removed: "ARM_Main_Ver8"

Commit message: ver9
Parts:
- added C11: 10u, Capacitor_THT:C_Disc_D5.1mm_W3.2mm_P5.00mm, F.Cu at (163.0, 61.0)
- added C12: 0.1u, Capacitor_THT:C_Disc_D5.1mm_W3.2mm_P5.00mm, F.Cu at (167.0, 61.0)
- added C13: 10u, Capacitor_THT:C_Disc_D5.1mm_W3.2mm_P5.00mm, F.Cu at (181.5, 61.5)
- added C14: 0.1u, Capacitor_THT:C_Disc_D5.1mm_W3.2mm_P5.00mm, F.Cu at (176.8, 61.5)
- added C15: 470u, Capacitor_THT:CP_Radial_D5.0mm_P2.50mm, F.Cu at (147.0, 122.5)
- added C16: 0.1u, Capacitor_THT:C_Disc_D5.1mm_W3.2mm_P5.00mm, F.Cu at (147.3, 117.5)
- added C17: 0.1u, Capacitor_THT:C_Disc_D5.1mm_W3.2mm_P5.00mm, F.Cu at (138.0, 68.0)
- added C18: 1000u, Capacitor_THT:CP_Radial_D10.0mm_P5.00mm, F.Cu at (129.5, 67.9)
- added C19: 0.1u, Capacitor_THT:C_Disc_D5.1mm_W3.2mm_P5.00mm, F.Cu at (115.0, 85.0)
- moved C8 37.4 mm to (143.8, 79.4), turned to 90 degrees
- moved SW4 32.9 mm to (114.5, 68.0), turned to 180 degrees
- moved U3 31.8 mm to (150.0, 79.5), turned to 180 degrees
- moved R1 26.7 mm to (129.0, 84.2), turned to 90 degrees
- moved J1 22.9 mm to (104.5, 90.5), turned to 90 degrees
- moved C9 22.6 mm to (155.8, 80.1), turned to 90 degrees
- moved U2 18.8 mm to (166.5, 90.0), turned to 180 degrees
- moved R4 14.7 mm to (132.5, 84.2)
- moved C2 14.2 mm to (136.5, 83.5)
- moved D2 14.1 mm to (136.5, 76.0)
- moved R5 14.1 mm to (140.5, 83.5)
- moved C10 12.7 mm to (115.4, 94.0)
- moved SB1 11.9 mm to (149.5, 72.5), turned to 90 degrees
- moved C1 11.7 mm to (125.0, 84.0)
- moved MD1 10.8 mm to (132.0, 92.0)
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Routing:
- net +5V_Analog: track 166.3 -> 135.6 mm, vias 4 -> 0
- net Net-(J2-Pin_2): track 8.43 -> 38.9 mm
- net Net-(U1-GPIO23/GPIO_GEN4): track 34.4 -> 5.45 mm
- net Net-(J3-Pin_2): track 9.21 -> 35.4 mm
- net Batte: track 95.5 -> 72.2 mm
- net Net-(J5-Pin_1): track 7.94 -> 28.2 mm
- net Net-(SB1-A1): track 31.0 -> 12.7 mm
- net Net-(U1-GPIO24/GPIO_GEN5): track 21.8 -> 6.12 mm
- net Net-(U1-3V3_1): track 37.7 -> 53.0 mm
- net Net-(IC2-ANODE): track 19.7 -> 6.08 mm, vias 1 -> 0
- net GNDA: track 93.5 -> 106.1 mm, vias 153 -> 156
- net Net-(SB1-Y2): track 22.7 -> 11.4 mm
- net +5V_Digital: track 67.2 -> 77.1 mm, vias 1 -> 0
- net Net-(U1-GPIO15/RXD0): track 13.1 -> 20.3 mm
- net Net-(IC2-COLLECTER): track 11.0 -> 17.7 mm
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Other:
- board size 99 x 78.5 mm -> 100 x 80 mm
- board text added: "ARM_Main_Ver9"
- board text removed: "ARM_Main_Ver8.1"

Commit message: ver9_add3dmodel
Parts:
- HS1: footprint heatsync:heatsink23.5_17_25mm -> Heatsync:heatsink23.5_17_25mm
- moved HS1 2.47 mm to (117.3, 121.3)
- moved VR1 1.37 mm to (117.5, 116.2)
Routing:
- net +5V_Analog: track 135.6 -> 137.0 mm
- net Net-(D4-A): track 24.3 -> 24.8 mm

Commit message: ver10
Parts:
- removed VR1: LM317T, Njm317_original:TO254P1054X470X1955-3
- added C12: 10u, Capacitor_THT:C_Disc_D5.1mm_W3.2mm_P5.00mm, F.Cu at (141.6, 71.2)
- added C16: 0.1u, Capacitor_THT:C_Disc_D5.1mm_W3.2mm_P5.00mm, F.Cu at (145.6, 71.2)
- added C17: 10u, Capacitor_THT:C_Disc_D5.1mm_W3.2mm_P5.00mm, F.Cu at (153.8, 102.2)
- added C18: 0.1u, Capacitor_THT:C_Disc_D5.1mm_W3.2mm_P5.00mm, F.Cu at (153.9, 74.4)
- added C19: 10u, Capacitor_THT:C_Disc_D5.1mm_W3.2mm_P5.00mm, F.Cu at (154.2, 92.2)
- added C21: 0.1u, Capacitor_THT:C_Disc_D5.1mm_W3.2mm_P5.00mm, F.Cu at (157.6, 102.2)
- added C22: 10u, Capacitor_THT:C_Disc_D5.1mm_W3.2mm_P5.00mm, F.Cu at (157.8, 74.5)
- added C23: 0.1u, Capacitor_THT:C_Disc_D5.1mm_W3.2mm_P5.00mm, F.Cu at (157.9, 92.0)
- added U4: LM350_TO220, Package_TO_SOT_THT:TO-220-3_Vertical, F.Cu at (120.1, 115.7)
- R4: renamed from R6; value 180 -> 120
- moved C13 5.09 mm to (142.8, 119.8), turned to 90 degrees
- moved SW3 4.36 mm to (153.2, 113.3)
- moved J3 4.33 mm to (149.2, 125.7)
- moved J4 4.06 mm to (154.4, 125.7)
- moved J5 3.95 mm to (159.3, 125.8)
- moved C10 3.80 mm to (137.4, 64.2), turned to -90 degrees
- moved C15 3.11 mm to (144.5, 124.2)
- moved IC2 2.88 mm to (164.5, 73.0)
- moved U2 2.59 mm to (168.7, 91.5)
- moved C20 1.81 mm to (155.6, 81.9)
- moved IC1 1.66 mm to (164.3, 98.3)
- moved C24 1.26 mm to (164.2, 60.6)
- moved C25 1.08 mm to (168.0, 60.6)
- moved J2 0.68 mm to (146.5, 61.8)
- moved RV2 0.56 mm to (140.5, 93.2)
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- renumbered C3 to C1, C17 to C10, C5 to C11, C16 to C13, C8 to C14, C4 to C2, C9 to C20, C11 to C24, C12 to C25, C14 to C26, C13 to C27, C19 to C3, C10 to C4, C7 to C5, C1 to C7, C18 to C8, C2 to C9, D3 to D1, D1 to D2, D4 to D3, D2 to D4, J5 to J2, J2 to J3, J3 to J4, J4 to J5, R2 to R1, R1 to R2, R4 to R3, R7 to R6, R3 to R7, RV2 to RV1, RV1 to RV2, SW4 to SW1, SW6 to SW2, SW5 to SW3, U3 to U1, U1 to U3
Routing:
- net +5V_Analog: track 137.0 -> 168.6 mm
- net GNDA: track 106.1 -> 122.8 mm, vias 156 -> 164
- net Net-(U1-VDD1): track 53.0 -> 64.7 mm
- net Net-(J3-Pin_1): track 29.8 -> 37.7 mm
- net +5V_Digital: track 77.1 -> 71.8 mm
- net Net-(U1-VOA): track 20.3 -> 23.7 mm
- net Net-(IC1-COLLECTER): track 24.4 -> 27.8 mm
- net Net-(J3-Pin_2): track 38.9 -> 41.9 mm
- net Net-(U3-GPIO23/GPIO_GEN4): track 5.45 -> 2.69 mm
- net Net-(IC2-COLLECTER): track 17.7 -> 20.1 mm, vias 0 -> 2
- net Net-(D5-A): track 9.43 -> 7.29 mm
- net Net-(J4-Pin_2): track 35.4 -> 37.0 mm
- net Net-(IC1-ANODE): track 9.77 -> 9.09 mm
- net Net-(MD1-TRIM): track 5.91 -> 5.31 mm
- net Net-(J2-Pin_1): track 28.2 -> 27.7 mm
Other:
- board text added: "ARM_Main_Ver10"
- board text removed: "ARM_Main_Ver9"

Commit message: ver10.1
Parts:
- moved C27 4.96 mm to (181.2, 66.5), turned to 90 degrees
- moved C14 1.05 mm to (143.9, 78.3)
Connections:
- C27 pad 1: GNDA -> Net-(U1-VDD1)
- C27 pad 2: Net-(U1-VDD1) -> GNDA
Routing:
- net +5V_Digital: track 71.8 -> 84.5 mm
- net Net-(U1-VDD1): track 64.7 -> 63.3 mm
- net +5V_Analog: track 168.6 -> 170.0 mm
- net Net-(SB1-A1): track 12.7 -> 13.4 mm
- net GNDA: track 122.8 -> 122.4 mm, vias 164 -> 172
Other:
- board text added: "ARM_Main_Ver10.1"
- board text removed: "ARM_Main_Ver10"

Commit message: ver10.1
Other:
- outline, holes or cut-outs redrawn
- board text added: "5V_A"
- board text added: "5V_D"
- board text added: "Batt"
Changed lines of the file:
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@@
 	(gr_circle
 		(center 102.5 130)
-		(end 104.6 130)
+		(end 104.2 130)
 		(stroke
 			(width 0.05)
@@
 	(gr_circle
 		(center 195 56)
-		(end 197.1 56)
+		(end 196.7 56)
 		(stroke
 			(width 0.05)
@@
 	(gr_circle
 		(center 102.5 56)
-		(end 104.6 56)
+		(end 104.2 56)
 		(stroke
 			(width 0.05)
@@
 	(gr_circle
 		(center 195 130)
-		(end 197.1 130)
+		(end 196.7 130)
 		(stroke
 			(width 0.05)
@@
 		(fill no)
 		(layer "Edge.Cuts")
+	)
+	(gr_text "Batt"
+		(at 119.95 73.7 0)
+		(layer "F.SilkS")
+		(effects
+			(font
+				(size 1 1)
+				(thickness 0.1)
+			)
+			(justify left bottom)
+		)
+	)
+	(gr_text "5V_D"
+		(at 130.74 72.34 0)
+		(layer "F.SilkS")
+		(effects
+			(font
+				(size 1 1)
+				(thickness 0.1)
+			)
+			(justify left bottom)
+		)
 	)
 	(gr_text "ARM_Main_Ver10.1"
@@
 			)
 			(justify left bottom)
+		)
+	)
+	(gr_text "5V_A"
+		(at 136.16 102.1 0)
+		(layer "F.SilkS")
+		(effects
+			(font
+				(size 1 1)
+				(thickness 0.1)
+			)
+			(justify left bottom)
