File: Arm_Main.kicad_sch (KiCad schematic)
At the start: 33 parts, among them IC1 TLP559_F_, J1 Conn_01x03_Socket, J2 Conn_01x02_Pin, J4 Conn_01x03_Pin, J5 Conn_01x03_Pin, J6 Conn_01x03_Pin, SW2 SW_SPDT, U1 RASPBERRY_PI_ZERO_2_W, U2 TLP2531, U3 TLP2531

Commit message: ver6
Connections:
- net GNDA: now also J1.2 (Pin_2), U1.18 (GPIO24/GPIO_GEN5), U2.4 (ANODE), U2.7 (VO1), U3.4 (ANODE)
- net at C1.1, C3.1, C4.1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: no longer SB1.8 (Vcc)
- net at U1.1 (3V3_1): now also SB1.8 (Vcc)
- net at SB1.7 (G), U1.12 (GPIO18/GPIO_GEN1): now also SB1.1 (G')
- net at U1.15 (GPIO22/GPIO_GEN3): no longer SB1.1 (G')
Other:
- note added: "3-Terminal Regulator"
- note added: "Krs"
- note added: "Sg90_connecter"
- note added: "Sg90_fotocapular"
- moved on the sheet: C3, C4, C5, C6, C7, D3, D4, HS1, J4, J5, J6, R6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

Commit message: Ver_7
Parts:
- removed C3, C6: 0.1u, Capacitor_THT:C_Disc_D5.1mm_W3.2mm_P5.00mm, symbol Device:C
- removed C4: 100u, Capacitor_THT:CP_Radial_D5.0mm_P2.50mm, symbol Device:C_Polarized
- removed C7: 47u, Capacitor_THT:CP_Radial_D5.0mm_P2.50mm, symbol Device:C_Polarized
- removed J1: Conn_01x03_Socket, Connector_JST:JST_XH_B3B-XH-A_1x03_P2.50mm_Vertical, symbol Connector:Conn_01x03_Socket
- removed J2: Conn_01x02_Pin, Connector_AMASS:AMASS_XT30U-F_1x02_P5.0mm_Vertical, symbol Connector:Conn_01x02_Pin
- removed J5, J6: Conn_01x03_Pin, Connector_PinHeader_2.54mm:PinHeader_1x03_P2.54mm_Vertical, symbol Connector:Conn_01x03_Pin
- removed SW2: SW_SPDT, Togle_original:TogleSW3pin, symbol Switch:SW_SPDT
- removed U3: TLP2531, U_DIP8_11-10C4S_TOS, symbol TLP2531_sym:TLP2531
- added C3: 100u, Capacitor_THT:CP_Radial_D5.0mm_P2.50mm, symbol Device:C_Polarized
- added C4, C7: 0.1u, Capacitor_THT:C_Disc_D5.1mm_W3.2mm_P5.00mm, symbol Device:C
- added C6: 47u, Capacitor_THT:CP_Radial_D5.0mm_P2.50mm, symbol Device:C_Polarized
- added D5: LED, LED_THT:LED_D3.0mm, symbol Device:LED
- added J1: Conn_01x02_Pin, Connector_AMASS:AMASS_XT30U-F_1x02_P5.0mm_Vertical, symbol Connector:Conn_01x02_Pin
- added J2, J3: Conn_01x03_Pin, Connector_PinHeader_2.54mm:PinHeader_1x03_P2.54mm_Vertical, symbol Connector:Conn_01x03_Pin
- added J5: Conn_01x03_Socket, Connector_JST:JST_XH_B3B-XH-A_1x03_P2.50mm_Vertical, symbol Connector:Conn_01x03_Socket
- added R7: 1k, Resistor_THT:R_Axial_DIN0207_L6.3mm_D2.5mm_P10.16mm_Horizontal, symbol Device:R
- added SW1: SW_SPDT, Togle_original:TogleSW3pin, symbol Switch:SW_SPDT
- added U3: ADuM121N, Package_SO:SOIC-8_3.9x4.9mm_P1.27mm, symbol Isolator:ADuM121N
- R1: value 20k -> 2k
- R2: value 1.2k -> 20k
- R4: value 2k -> 1.2k
- RV1, RV2: value R_Potentiometer_Trim -> R_Trim
- U2: footprint ul_TLP2531:U_DIP8_11-10C4S_TOS -> U_DIP8_11-10C4S_TOS
- VR1: footprint NJM317:TO254P1054X470X1955-3 -> Njm317_original:TO254P1054X470X1955-3
Connections:
- net GNDA: now also R4.2, C3.2, C4.2, C6.2, C7.2, D5.1 (K), J1.1 (Pin_1), J2.3 (Pin_3), J3.3 (Pin_3), J5.3 (Pin_3), U3.4 (GND1), U3.5 (GND2); no longer R1.2, U1.18 (GPIO24/GPIO_GEN5), U2.4 (ANODE), U2.7 (VO1)
- net Batte: now reaches C1.1, D3.1 (K), IC1.8 (VCC), MD1.2 (VIN), R1.1, U2.8 (VCC), VR1.3 (VIN)
- net Batte: now also R2.1, C3.1, C4.1, J5.1 (Pin_1), SW1.1 (A); no longer R4.1
- net at D1.2 (A): now also R1.2; no longer R4.2
- net +5V_Digital: now reaches C2.1, MD1.4 (VOUT), MD1.5 (SENSE), R5.1, U1.2 (5V_2)
- net +5V_Digital: now also R4.1, U1.4 (5V_4); no longer R2.1
- net at U1.16 (GPIO23/GPIO_GEN4): now also U2.4 (ANODE)
- net at J4.2 (Pin_2): now also IC1.6 (COLLECTER)
- net at SB1.8 (Vcc), U1.1 (3V3_1): now also U1.17 (3V3_17), U3.1 (VDD1)
- net at SB1.1 (G'), SB1.7 (G): now also U1.13 (GPIO27/GPIO_GEN2); no longer U1.12 (GPIO18/GPIO_GEN1)
- net at SB1.2 (A1), SB1.3 (Y2): now also U1.12 (GPIO18/GPIO_GEN1); no longer U1.13 (GPIO27/GPIO_GEN2)
- net +5V_Analog: now reaches D3.2 (A), D4.1 (K), J4.1 (Pin_1), R6.2, VR1.2 (VOUT)
- net +5V_Analog: now also C6.1, C7.1, J2.1 (Pin_1), J3.1 (Pin_1), R7.1, U3.8 (VDD2)
- net at SB1.5 (A2), SB1.6 (Y1): now also U3.2 (VOA), U3.3 (VIB); no longer U2.1 (ANODE), U2.6 (VO2)
- new net: J2.2 (Pin_2), U2.6 (VO2)
- new net: J3.2 (Pin_2), U2.7 (VO1)
- new net: J1.2 (Pin_2), SW1.2 (B)
- new net: U1.18 (GPIO24/GPIO_GEN5), U2.1 (ANODE)
- new net: J5.2 (Pin_2), U3.6 (VOB), U3.7 (VIA)
- new net: D5.2 (A), R7.2
Other:
- note added: "DCDC_Converter"
- note added: "Isoleter"
- note added: "To_KRS_Servo"
- note added: "To_SG90_Servo"
- note removed: "Krs"
- note removed: "Sg90_connecter"
- note removed: "Sg90_fotocapular"

Commit message: ver.8.pre
Parts:
- removed SW1: SW_SPDT, Togle_original:TogleSW3pin, symbol Switch:SW_SPDT
- added C10: 1000u, Capacitor_THT:CP_Radial_D10.0mm_P5.00mm, symbol Device:C_Polarized
- added C8, C9: 0.1u, Capacitor_THT:C_Disc_D5.1mm_W3.2mm_P5.00mm, symbol Device:C
- added IC2: TLP559_F_, TLP559:DIP762W60P254L966H485Q8N, symbol tlp559:TLP559_F_
- added SW4, SW5, SW6: SW_SPST, Togle_original:Hadou_Sw, symbol Switch:SW_SPST
Connections:
- net +5V_Analog: now also IC1.8 (VCC), SB1.8 (Vcc), U2.8 (VCC), IC2.8 (VCC), SW5.1 (A); no longer J2.1 (Pin_1), J3.1 (Pin_1), J4.1 (Pin_1)
- net Batte: now also C10.1, SW4.2 (B), SW6.2 (B); no longer IC1.8 (VCC), J5.1 (Pin_1), U2.8 (VCC)
- net GNDA: now also C10.2, IC2.3 (CATHODE), IC2.5 (EMITTER)
- net at SB1.1 (G'), SB1.7 (G): now also IC2.6 (COLLECTER); no longer U1.13 (GPIO27/GPIO_GEN2)
- net at SB1.5 (A2), SB1.6 (Y1): now also J5.2 (Pin_2); no longer U3.2 (VOA), U3.3 (VIB)
- net at U1.1 (3V3_1), U1.17 (3V3_17), U3.1 (VDD1): no longer SB1.8 (Vcc)
- net at J1.2 (Pin_2): now also SW6.1 (A)
- net at U1.10 (GPIO15/RXD0): now also U3.2 (VOA), C9.1
- net at U1.36 (GPIO16): now also IC2.2 (ANODE)
- net at U1.8 (GPIO14/TXD0): now also U3.3 (VIB), C9.2
- new net: J5.1 (Pin_1), SW4.1 (A)
- new net: C8.2, SB1.2 (A1), U3.6 (VOB)
- new net: C8.1, SB1.3 (Y2), U3.7 (VIA)
- new net: J2.1 (Pin_1), J3.1 (Pin_1), J4.1 (Pin_1), SW5.2 (B)
- now unconnected: U1.12 (GPIO18/GPIO_GEN1)
Other:
- moved on the sheet: IC1, J5, SB1, U2, U3

Commit message: v8.1
Connections:
- net at IC2.2 (ANODE): now also U1.12 (GPIO18/GPIO_GEN1); no longer U1.36 (GPIO16)
Changed lines of the file:
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@@
-	(wire
-		(pts
-			(xy 91.44 105.41) (xy 91.44 123.19)
-		)
-		(stroke
-			(width 0)
-			(type default)
-		)
-	)
 	(wire
 		(pts
@@
 	(wire
 		(pts
-			(xy 76.2 90.17) (xy 82.55 90.17)
-		)
-		(stroke
-			(width 0)
-			(type default)
-		)
-	)
-	(wire
-		(pts
 			(xy 45.72 21.59) (xy 54.61 21.59)
 		)
@@
 	(wire
 		(pts
-			(xy 82.55 90.17) (xy 82.55 105.41)
-		)
-		(stroke
-			(width 0)
-			(type default)
-		)
-	)
-	(wire
-		(pts
 			(xy 201.93 39.37) (xy 201.93 43.18)
 		)
@@
 	(wire
 		(pts
-			(xy 82.55 105.41) (xy 91.44 105.41)
-		)
-		(stroke
-			(width 0)
-			(type default)
-		)
-	)
-	(wire
-		(pts
 			(xy 54.61 54.61) (xy 54.61 62.23)
 		)
@@
 	(wire
 		(pts
+			(xy 76.2 95.25) (xy 78.74 95.25)
+		)
+		(stroke
+			(width 0)
+			(type default)
+		)
+	)
+	(wire
+		(pts
 			(xy 24.13 31.75) (xy 24.13 26.67)
 		)
@@
 	(wire
 		(pts
+			(xy 78.74 102.87) (xy 91.44 102.87)
+		)
+		(stroke
+			(width 0)
+			(type default)
+		)
+	)
+	(wire
+		(pts
 			(xy 123.19 54.61) (xy 139.7 54.61)
 		)
@@
 	(wire
 		(pts
+			(xy 78.74 95.25) (xy 78.74 102.87)
+		)
+		(stroke
+			(width 0)
+			(type default)
+		)
+	)
+	(wire
+		(pts
 			(xy 148.59 144.78) (xy 148.59 127)
 		)
@@
 		)
 		(stroke
+			(width 0)
+			(type default)
+		)
+	)
+	(wire
+		(pts
+			(xy 91.44 102.87) (xy 91.44 123.19)
+		)
+		(stroke

Commit message: ver9
Parts:
- added C11, C13: 10u, Capacitor_THT:C_Disc_D5.1mm_W3.2mm_P5.00mm, symbol Device:C
- added C12, C14, C16, C17, C19: 0.1u, Capacitor_THT:C_Disc_D5.1mm_W3.2mm_P5.00mm, symbol Device:C
- added C15: 470u, Capacitor_THT:CP_Radial_D5.0mm_P2.50mm, symbol Device:C_Polarized
- added C18: 1000u, Capacitor_THT:CP_Radial_D10.0mm_P5.00mm, symbol Device:C_Polarized
Connections:
- net +5V_Digital: now also C11.2, C12.2
- net Batte: now also C19.1
- net GNDA: now also C11.1, C12.1, C13.1, C14.1, C15.2, C16.2, C17.2, C18.2, C19.2
- net at J5.1 (Pin_1), SW4.1 (A): now also C17.1, C18.1
- net at J2.1 (Pin_1), J3.1 (Pin_1), J4.1 (Pin_1)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: now also C15.1, C16.1
- net at U1.1 (3V3_1), U1.17 (3V3_17), U3.1 (VDD1): now also C13.2, C14.2
Other:
- moved on the sheet: SW4, SW5

Commit message: ver9_add3dmodel
Parts:
- HS1: footprint heatsync:heatsink23.5_17_25mm -> Heatsync:heatsink23.5_17_25mm
Changed lines of the file:
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@@
 	(title_block
 		(title "ARM_Main")
-		(date "2025-09-03")
+		(date "2025-09-30")
+		(rev "ver9")
 		(company "Takuya Kamada")
 	)
@@
 	(wire
 		(pts
-			(xy 101.6 76.2) (xy 101.6 80.01)
+			(xy 101.6 74.93) (xy 101.6 80.01)
 		)
 		(stroke
@@
 	(wire
 		(pts
-			(xy 88.9 74.93) (xy 83.82 74.93)
+			(xy 86.36 74.93) (xy 83.82 74.93)
 		)
 		(stroke
@@
 	(global_label "+5V_Digital"
 		(shape output)
-		(at 88.9 74.93 0)
+		(at 86.36 74.93 0)
 		(fields_autoplaced yes)
 		(effects
@@
 		)
 		(property "Intersheetrefs" "${INTERSHEET_REFS}"
-			(at 102.8918 74.93 0)
+			(at 100.3518 74.93 0)
 			(effects
 				(font
@@
 	(global_label "+5V_Analog"
 		(shape output)
-		(at 101.6 76.2 90)
+		(at 101.6 74.93 0)
 		(fields_autoplaced yes)
 		(effects
@@
 		)
 		(property "Intersheetrefs" "${INTERSHEET_REFS}"
-			(at 101.6 62.0269 90)
+			(at 115.7731 74.93 0)
 			(effects
 				(font
@@
 			)
 		)
-		(property "Footprint" "heatsync:heatsink23.5_17_25mm"
+		(property "Footprint" "Heatsync:heatsink23.5_17_25mm"
 			(at 216.8652 52.07 0)
 			(effects

Commit message: ver10
Parts:
- removed VR1: LM317T, Njm317_original:TO254P1054X470X1955-3, symbol LM317T:LM317T
- added C12, C17, C19, C22: 10u, Capacitor_THT:C_Disc_D5.1mm_W3.2mm_P5.00mm, symbol Device:C
- added C16, C18, C21, C23: 0.1u, Capacitor_THT:C_Disc_D5.1mm_W3.2mm_P5.00mm, symbol Device:C
- added U4: LM350_TO220, Package_TO_SOT_THT:TO-220-3_Vertical, symbol Regulator_Linear:LM350_TO220
- R4: renamed from R6; value 180 -> 120
- U2: footprint U_DIP8_11-10C4S_TOS -> ul_TLP2531:U_DIP8_11-10C4S_TOS
- renumbered C3 to C1, C17 to C10, C5 to C11, C16 to C13, C8 to C14, C4 to C2, C9 to C20, C11 to C24, C12 to C25, C14 to C26, C13 to C27, C19 to C3, C10 to C4, C7 to C5, C1 to C7, C18 to C8, C2 to C9, D3 to D1, D1 to D2, D4 to D3, D2 to D4, J5 to J2, J2 to J3, J3 to J4, J4 to J5, R2 to R1, R1 to R2, R4 to R3, R7 to R6, R3 to R7, RV2 to RV1, RV1 to RV2, SW4 to SW1, SW6 to SW2, SW5 to SW3, U3 to U1, U1 to U3
Connections:
- net +5V_Analog: now also C12.1, C16.1, C17.1, C18.1, C19.1, C21.1, C22.1, C23.1, U4.2 (VO)
- net Batte: now also U4.3 (VI)
- net GNDA: now also C12.2, C16.2, C17.2, C18.2, C19.2, C21.2, C22.2, C23.2
- net at C11.1, D3.2 (A), R4.1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: now also U4.1 (ADJ)
Other:
- moved on the sheet: C13, C15, J3, J4, J5, SW3

Commit message: ver10.1
Connections:
- net GNDA: now also C27.2; no longer C27.1
- net at C26.2, U1.1 (VDD1), U3.1 (3V3_1)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: now also C27.1; no longer C27.2
Other:
- moved on the sheet: C10, C12, C13, C14, C15, C16, C17, C18, C19, C20, C21, C22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
